File: digitalSystemChipBoard.kicad_pcb (KiCad board)
At the start: 4 copper layers, 32 x 32 mm, 14 parts, among them J0 Conn_01x10_Female, J1 Conn_01x10_Female, J2 Conn_01x10_Female, J3 Conn_01x10_Female, U0 ATmega1284P-AU, U1 CH340B, U2 ICSP, Y0 16MHz

Commit message: Edit some track
Routing:
- net GND: track 111.5 -> 108.8 mm
- net /ADJUST_CLK: track 24.4 -> 25.6 mm
- net /MOSI: track 49.4 -> 50.0 mm
- net /SCK: track 30.1 -> 29.6 mm
